Commit message: revise walker robot urdf

File: assets/walker/urdf/walker_tienkung_ei_nofinger.urdf (robot description, URDF)
Before this commit: robot humanoid, 60 links, 59 joints
Links:
- removed link L_base_link
- removed link R_base_link
- removed link camera_body_back_link
- removed link camera_body_front_link
- removed link camera_head_link
- removed link left_index_1
- removed link left_index_2
- removed link left_little_1
- removed link left_little_2
- removed link left_middle_1
- removed link left_middle_2
- removed link left_ring_1
- removed link left_ring_2
- removed link left_thumb_1
- removed link left_thumb_2
- removed link left_thumb_3
- removed link left_thumb_4
- removed link right_index_1
- removed link right_index_2
- removed link right_little_1
- removed link right_little_2
- removed link right_middle_1
- removed link right_middle_2
- removed link right_ring_1
- removed link right_ring_2
- removed link right_thumb_1
- removed link right_thumb_2
- removed link right_thumb_3
- removed link right_thumb_4
- added link imu, mass 0.02; collision mesh filename=meshes/imu_link.STL; visual mesh filename=meshes/imu_link.STL
- added link left_tcp_link, mass 0.218186; collision mesh filename=meshes/left_tcp_link.STL; visual mesh filename=meshes/left_tcp_link.STL
- added link ob_camera_back_link, mass 0.1; collision mesh filename=meshes/camera_body_back_link.STL; visual mesh filename=meshes/camera_body_back_link.STL
- added link ob_camera_head_link, mass 0.1; collision mesh filename=meshes/camera_head_link.STL; visual mesh filename=meshes/camera_head_link.STL
- added link ob_camera_waist_link, mass 0.1; collision mesh filename=meshes/camera_body_front_link.STL; visual mesh filename=meshes/camera_body_front_link.STL
- added link right_tcp_link, mass 0.218186; collision mesh filename=meshes/right_tcp_link.STL; visual mesh filename=meshes/right_tcp_link.STL
- link elbow_pitch_l_link: mass 0.222661 -> 0.246311
- link elbow_pitch_r_link: mass 0.222661 -> 0.246311
- link elbow_yaw_l_link: mass 0.990079 -> 0.986828
- link elbow_yaw_r_link: mass 0.990079 -> 0.986828
- link head_pitch_link: mass 0.230460 -> 0.23046
- link head_yaw_link: mass 0.0883927289639252 -> 0.088397
- link hip_pitch_l_link: mass 4.227933 -> 3.951912
- link hip_pitch_r_link: mass 4.227933 -> 3.951912
- link hip_yaw_l_link: mass 6.572700 -> 6.670795
- link hip_yaw_r_link: mass 7.182896 -> 6.670795
- link knee_pitch_l_link: mass 3.017992 -> 2.312685
- link knee_pitch_r_link: mass 3.017992 -> 2.312685
- link pelvis: mass 6.094610 -> 5.639
- link shoulder_pitch_l_link: mass 1.030628 -> 1.032698
- link shoulder_pitch_r_link: mass 1.030628 -> 1.032698
- link shoulder_roll_l_link: mass 0.412600522097283 -> 0.440997
- link shoulder_roll_r_link: mass 0.412600522097283 -> 0.440997
- link shoulder_yaw_l_link: mass 1.307604 -> 1.365033
- link shoulder_yaw_r_link: mass 1.307604 -> 1.365033
- link waist_yaw_link: mass 22.445155 -> 22.0
- link wrist_pitch_l_link: mass 0.266415 -> 0.262007
- link wrist_pitch_r_link: mass 0.266415 -> 0.262007
- link wrist_roll_l_link: mass 0.065684 -> 0.131751
- link wrist_roll_r_link: mass 0.065684 -> 0.131751
Joints:
- removed joint left_hand_joint
- removed joint left_index_1_joint
- removed joint left_index_2_joint
- removed joint left_little_1_joint
- removed joint left_little_2_joint
- removed joint left_middle_1_joint
- removed joint left_middle_2_joint
- removed joint left_ring_1_joint
- removed joint left_ring_2_joint
- removed joint left_thumb_1_joint
- removed joint left_thumb_2_joint
- removed joint left_thumb_3_joint
- removed joint left_thumb_4_joint
- removed joint right_hand_joint
- removed joint right_index_1_joint
- removed joint right_index_2_joint
- removed joint right_little_1_joint
- removed joint right_little_2_joint
- removed joint right_middle_1_joint
- removed joint right_middle_2_joint
- removed joint right_ring_1_joint
- removed joint right_ring_2_joint
- removed joint right_thumb_1_joint
- removed joint right_thumb_2_joint
- removed joint right_thumb_3_joint
- removed joint right_thumb_4_joint
- removed joint waist_yaw_joint
- added joint body_yaw_joint: type revolute, parent pelvis, child waist_yaw_link, origin xyz=0 0 0 rpy=0 0 0, axis 0 0 1, limit lower=-2.9670597283903604 upper=3.141592653589793 effort=91.0 velocity=9.215338450530059
- added joint imu_joint: type fixed, parent pelvis, child imu, origin xyz=0.0499 -0.0358 -0.03194 rpy=0 0 0, axis 0 0 0
- added joint left_tcp_joint: type fixed, parent wrist_roll_l_link, child left_tcp_link, origin xyz=0 0 -0.0848 rpy=0 0 0, axis 0 0 0
- added joint right_tcp_joint: type fixed, parent wrist_roll_r_link, child right_tcp_link, origin xyz=0 0 -0.0848 rpy=0 0 0, axis 0 0 0
- joint ankle_pitch_l_joint: limit lower=-1.22 upper=0.5236 effort=60 velocity=12.8 -> lower=-1.2217304763960306 upper=0.5235987755982988 effort=55.0 velocity=14.137166941154069
- joint ankle_pitch_r_joint: limit lower=-1.22 upper=0.5236 effort=60 velocity=12.8 -> lower=-1.2217304763960306 upper=0.5235987755982988 effort=55.0 velocity=14.137166941154069; origin xyz=0 0.00074981 -0.4 rpy=0 0 0 -> xyz=0 0.00099989 -0.4 rpy=0 0 0
- joint ankle_roll_l_joint: limit lower=-0.4363 upper=0.4363 effort=30 velocity=7.8 -> lower=-0.5235987755982988 upper=0.5235987755982988 effort=55.0 velocity=14.137166941154069
- joint ankle_roll_r_joint: limit lower=-0.4363 upper=0.4363 effort=30 velocity=7.8 -> lower=-0.5235987755982988 upper=0.5235987755982988 effort=55.0 velocity=14.137166941154069
- joint camera_body_back_joint: child camera_body_back_link -> ob_camera_back_link; origin xyz=-0.1054 0 0.29423 rpy=-3.1416 0.43633 -3.1416 -> xyz=-0.11363 0.02375 0.2746 rpy=2.0071 0 -1.5708
- joint camera_body_front_joint: child camera_body_front_link -> ob_camera_waist_link; origin xyz=0.06958 0 0.035588 rpy=0 0.57596 0 -> xyz=0.090583 0.02375 0.039012 rpy=-2.1468 0 -1.5708
- joint camera_head_joint: child camera_head_link -> ob_camera_head_link; origin xyz=0.052782 -6.5455E-05 0.067499 rpy=0 0.2618 0 -> xyz=0.075191 0.010935 0.074436 rpy=-1.8326 0 -1.5708
- joint elbow_pitch_l_joint: limit lower=-2.61 upper=0.261 effort=30 velocity=7.3 -> lower=-2.6179938779914944 upper=0.2617993877991494 effort=35.0 velocity=5.235987755982989
- joint elbow_pitch_r_joint: limit lower=-2.61 upper=0.261 effort=30 velocity=7.3 -> lower=-2.6179938779914944 upper=0.2617993877991494 effort=35.0 velocity=5.235987755982989
- joint elbow_yaw_l_joint: limit lower=-2.9671 upper=2.9671 effort=15 velocity=14.6 -> lower=-2.9670597283903604 upper=2.9670597283903604 effort=24.0 velocity=10.471975511965978
- joint elbow_yaw_r_joint: limit lower=-2.9671 upper=2.9671 effort=15 velocity=14.6 -> lower=-2.9670597283903604 upper=2.9670597283903604 effort=24.0 velocity=10.471975511965978
- joint head_pitch_joint: limit lower=-0.43 upper=0.43 effort=9 velocity=7.2 -> lower=-0.4363323129985824 upper=0.4363323129985824 effort=6.3 velocity=7.5398223686155035
- joint head_roll_joint: limit lower=-0.43 upper=0.43 effort=9 velocity=7.2 -> lower=-0.4537856055185257 upper=0.4537856055185257 effort=6.3 velocity=7.5398223686155035
- joint head_yaw_joint: limit lower=-1.57 upper=1.57 effort=9 velocity=7.2 -> lower=-1.5707963267948966 upper=1.5707963267948966 effort=6.3 velocity=7.5398223686155035
- joint hip_pitch_l_joint: limit lower=-2.79 upper=2.09 effort=300 velocity=12.5 -> lower=-2.792526803190927 upper=2.0943951023931953 effort=330.0 velocity=15.707963267948966
- joint hip_pitch_r_joint: limit lower=-2.79 upper=2.09 effort=300 velocity=12.5 -> lower=-2.792526803190927 upper=2.0943951023931953 effort=330.0 velocity=15.707963267948966
- joint hip_roll_l_joint: limit lower=-0.79 upper=0.79 effort=160 velocity=15.6 -> lower=-0.7853981633974483 upper=0.7853981633974483 effort=235.0 velocity=16.755160819145562
- joint hip_roll_r_joint: limit lower=-0.79 upper=0.79 effort=160 velocity=15.6 -> lower=-0.7853981633974483 upper=0.7853981633974483 effort=235.0 velocity=16.755160819145562
- joint hip_yaw_l_joint: limit lower=-1.04 upper=1.04 effort=160 velocity=15.6 -> lower=-1.0471975511965976 upper=1.0471975511965976 effort=235.0 velocity=16.755160819145562; origin xyz=0 0 -0.0987 rpy=0 0 0 -> xyz=0 -0.00015 -0.0987 rpy=0 0 0
- joint hip_yaw_r_joint: limit lower=-1.04 upper=1.04 effort=160 velocity=15.6 -> lower=-1.0471975511965976 upper=1.0471975511965976 effort=235.0 velocity=16.755160819145562
- joint knee_pitch_l_joint: limit lower=0.0 upper=2.39 effort=300 velocity=12.5 -> lower=0.0 upper=2.3911010752322315 effort=330.0 velocity=15.707963267948966; origin xyz=0 -4.2833E-05 -0.3013 rpy=0 0 0 -> xyz=0 0.00010715 -0.3013 rpy=0 0 0
- joint knee_pitch_r_joint: limit lower=0.0 upper=2.39 effort=300 velocity=12.5 -> lower=0.0 upper=2.3911010752322315 effort=330.0 velocity=15.707963267948966; origin xyz=0 0.00015001 -0.3013 rpy=0 0 0 -> xyz=0 9.9938E-05 -0.3013 rpy=0 0 0
- joint shoulder_pitch_l_joint: limit lower=-2.96 upper=2.96 effort=91 velocity=8.8 -> lower=-2.9670597283903604 upper=2.9670597283903604 effort=91.0 velocity=9.215338450530059; origin xyz=0 0.14539 0.37721 rpy=0.087266 0 0 -> xyz=0 0.1444 0.37712 rpy=0.087266 0 0
- joint shoulder_pitch_r_joint: limit lower=-2.96 upper=2.96 effort=91 velocity=8.8 -> lower=-2.9670597283903604 upper=2.9670597283903604 effort=91.0 velocity=9.215338450530059; origin xyz=0 -0.14539 0.37721 rpy=-0.087266 0 0 -> xyz=0 -0.1444 0.37712 rpy=-0.087266 0 0
- joint shoulder_roll_l_joint: limit lower=-0.2618 upper=3.4 effort=60 velocity=12 -> lower=-0.2617993877991494 upper=2.6179938779914944 effort=95.0 velocity=3.979350694547071
- joint shoulder_roll_r_joint: limit lower=-3.4 upper=0.2618 effort=60 velocity=12 -> lower=-2.6179938779914944 upper=0.2617993877991494 effort=95.0 velocity=3.979350694547071
- joint shoulder_yaw_l_joint: limit lower=-2.96 upper=2.96 effort=30 velocity=7.3 -> lower=-2.9670597283903604 upper=2.9670597283903604 effort=35.0 velocity=5.235987755982989
- joint shoulder_yaw_r_joint: limit lower=-2.96 upper=2.96 effort=30 velocity=7.3 -> lower=-2.9670597283903604 upper=2.9670597283903604 effort=35.0 velocity=5.235987755982989
- joint wrist_pitch_l_joint: limit lower=-1.3 upper=1.65 effort=9 velocity=7.2 -> lower=-0.7853981633974483 upper=1.0471975511965976 effort=6.3 velocity=7.5398223686155035; origin xyz=0 0.002 -0.1887 rpy=0 0 0 -> xyz=0 0 -0.1887 rpy=0 0 0
- joint wrist_pitch_r_joint: limit lower=-1.3 upper=1.65 effort=9 velocity=7.2 -> lower=-0.7853981633974483 upper=1.0471975511965976 effort=6.3 velocity=7.5398223686155035; origin xyz=0 -0.002 -0.1887 rpy=0 0 0 -> xyz=0 0 -0.1887 rpy=0 0 0
- joint wrist_roll_l_joint: limit lower=-1.04 upper=0.785 effort=9 velocity=7.2 -> lower=-1.6580627893946132 upper=1.3089969389957472 effort=6.3 velocity=7.5398223686155035; origin xyz=5.0485E-05 0 -0.02 rpy=0 0 0 -> xyz=0 0 -0.02 rpy=0 0 0
- joint wrist_roll_r_joint: limit lower=-1.04 upper=0.785 effort=9 velocity=7.2 -> lower=-1.3089969389957472 upper=1.6580627893946132 effort=6.3 velocity=7.5398223686155035; origin xyz=5.0485E-05 0 -0.02 rpy=0 0 0 -> xyz=0 0 -0.02 rpy=0 0 0
